Commit message: fix initialState if no rosparam is set

File: ocs2_robotic_assets/resources/tiago/urdf/tiago.urdf (robot description, URDF)
Before this commit: robot tiago, 19 links, 18 joints
Links:
- link base_link: geometry collision cylinder length=0.28 radius=0.265; visual mesh filename=package://pmb2_description/meshes/base/base.stl

Commit message: tiago urdf and collisions

File: ocs2_robotic_assets/resources/tiago/urdf/tiago.urdf (robot description, URDF)
Before this commit: robot tiago, 19 links, 18 joints
Links:
- added link suspension_left_link, mass 10
- added link suspension_right_link, mass 10
- added link wheel_left_link, mass 1.82362; collision sphere radius=0.0985; visual mesh filename=package://pmb2_description/meshes/wheels/wheel.stl
- added link wheel_right_link, mass 1.82362; collision sphere radius=0.0985; visual mesh filename=package://pmb2_description/meshes/wheels/wheel.stl
- link arm_1_link: geometry visual mesh filename=package://tiago_description/meshes/arm/arm_1.stl scale=1 1 1
- link arm_2_link: geometry visual mesh filename=package://tiago_description/meshes/arm/arm_2.stl scale=1 1 1
- link arm_3_link: geometry visual mesh filename=package://tiago_description/meshes/arm/arm_3.stl scale=1 1 1
- link arm_4_link: geometry visual mesh filename=package://tiago_description/meshes/arm/arm_4.stl scale=1 1 1
- link arm_5_link: geometry visual mesh filename=package://tiago_description/meshes/arm/arm_5-wrist-2017.stl scale=1 1 1
- link arm_6_link: geometry visual mesh filename=package://tiago_description/meshes/arm/arm_6-wrist-2017.stl scale=1 1 1
- link arm_tool_link: geometry collision cylinder length=0.2 radius=0.05; visual cylinder length=0.005 radius=0.005
- link hand_palm_link: geometry visual mesh filename=package://hey5_description/meshes/palm.stl scale=1 1 1
- link hand_thumb_link: geometry visual sphere radius=0.001
- link head_1_link: geometry visual mesh filename=package://tiago_description/meshes/head/head_1.stl scale=1 1 1
- link head_2_link: geometry collision box size=0.2 0.2 0.25; visual mesh filename=package://tiago_description/meshes/head/head_2.stl scale=1 1 1
- link torso_lift_link: geometry collision box size=0.25 0.25 0.45; visual mesh filename=package://tiago_description/meshes/torso/torso_lift_with_ar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 scale=1 1 1
Joints:
- added joint suspension_left_joint: type fixed, parent base_link, child suspension_left_link, origin xyz=0 0 0 rpy=0 0 0, axis 0 0 1, limit lower=-0.005 upper=0.005 effort=100.0 velocity=1.0
- added joint suspension_right_joint: type fixed, parent base_link, child suspension_right_link, origin xyz=0 0 0 rpy=0 0 0, axis 0 0 1, limit lower=-0.005 upper=0.005 effort=100.0 velocity=1.0
- added joint wheel_left_joint: type fixed, parent suspension_left_link, child wheel_left_link, origin xyz=0 0.2022 0.0 rpy=-1.57079632679 0 0, axis 0 0 1, limit effort=6.0 velocity=10.152284264
- added joint wheel_right_joint: type fixed, parent suspension_right_link, child wheel_right_link, origin xyz=0 -0.2022 0.0 rpy=-1.57079632679 0 0, axis 0 0 1, limit effort=6.0 velocity=10.152284264
