Commit message: hsr, update limits

File: ocs2_robotic_assets/resources/hsr/urdf/hsr.urdf (robot description, URDF)
Before this commit: robot hsrb, 24 links, 23 joints
Links:
- added link myfakepalmlink
Joints:
- added joint myfakejoint: type fixed, parent hand_palm_link, child myfakepalmlink, origin xyz=0.0 0.0 0.0 rpy=3.1415927 -1.5707963 0
- joint torso_lift_joint: type prismatic -> fixed
