Commit message: simplify pr2 collisions

File: ocs2_robotic_assets/resources/pr2/urdf/pr2.urdf (robot description, URDF)
Before this commit: robot pr2, 12 links, 11 joints
Links:
- link base_link: geometry collision box size=0.65 0.65 0.2; visual mesh filename=package://pr2_description/meshes/base_v0/base.dae
- link r_gripper_palm_link: geometry collision box size=0.1 0.1 0.1; visual mesh filename=package://pr2_description/meshes/gripper_v0/gripper_palm.dae
- link torso_lift_link: geometry collision box size=0.3 0.6 0.8; visual mesh filename=package://pr2_description/meshes/torso_v0/torso_lift.dae

Commit message: add head and fingers

File: ocs2_robotic_assets/resources/pr2/urdf/pr2.urdf (robot description, URDF)
Before this commit: robot pr2, 12 links, 11 joints
Links:
- added link head_pan_link, mass 6.339; visual mesh filename=package://pr2_description/meshes/head_v0/head_pan.dae
- added link head_tilt_link, mass 4.479; collision box size=0.27 0.28 0.27; visual mesh filename=package://pr2_description/meshes/head_v0/head_tilt.dae
- added link r_gripper_l_finger_link, mass 0.17126; visual mesh filename=package://pr2_description/meshes/gripper_v0/l_finger.dae
- added link r_gripper_r_finger_link, mass 0.17389; visual mesh filename=package://pr2_description/meshes/gripper_v0/l_finger.dae
- link r_elbow_flex_link: geometry visual mesh filename=package://pr2_description/meshes/upper_arm_v0/elbow_flex.dae
- link r_forearm_link: geometry collision box size=0.21 0.075 0.075; visual mesh filename=package://pr2_description/meshes/forearm_v0/forearm.dae
- link r_forearm_roll_link: geometry visual mesh filename=package://pr2_description/meshes/upper_arm_v0/forearm_roll.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
- link r_gripper_palm_link: geometry collision box size=0.08 0.095 0.065; visual mesh filename=package://pr2_description/meshes/gripper_v0/gripper_palm.dae
- link r_shoulder_lift_link: geometry visual mesh filename=package://pr2_description/meshes/shoulder_v0/shoulder_lift.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
- link r_shoulder_pan_link: geometry visual mesh filename=package://pr2_description/meshes/shoulder_v0/shoulder_pan.d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
- link r_upper_arm_link: geometry visual mesh filename=package://pr2_description/meshes/upper_arm_v0/upper_arm.dae
- link r_upper_arm_roll_link: geometry visual mesh filename=package://pr2_description/meshes/shoulder_v0/upper_arm_roll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
- link r_wrist_flex_link: geometry visual mesh filename=package://pr2_description/meshes/forearm_v0/wrist_flex.dae
- link r_wrist_roll_link: geometry collision box size=0.075 0.075 0.065; visual mesh filename=package://pr2_description/meshes/forearm_v0/wrist_roll.stl
Joints:
- added joint head_pan_joint: type fixed, parent torso_lift_link, child head_pan_link, origin xyz=-0.01707 0.0 0.38145 rpy=0.0 0.0 0.0, axis 0 0 1, limit lower=-3.007 upper=3.007 effort=2.645 velocity=6
- added joint head_tilt_joint: type fixed, parent head_pan_link, child head_tilt_link, origin xyz=0.068 0 0 rpy=0 0 0, axis 0 1 0, limit lower=-0.471238 upper=1.39626 effort=18 velocity=5
- added joint r_gripper_l_finger_joint: type fixed, parent r_gripper_palm_link, child r_gripper_l_finger_link, origin xyz=0.07691 0.01 0 rpy=0 0 0, axis 0 0 1, limit lower=0.0 upper=0.548 effort=1000.0 velocity=0.5
- added joint r_gripper_r_finger_joint: type fixed, parent r_gripper_palm_link, child r_gripper_r_finger_link, origin xyz=0.07691 -0.01 0 rpy=0 0 0, axis 0 0 -1, limit lower=0.0 upper=0.548 effort=1000.0 velocity=0.5, mimic joint=r_gripper_l_finger_joint multiplier=1 offset=0
- joint r_wrist_roll_joint: type continuous -> revolute

Commit message: colllision constraint v1

File: ocs2_robotic_assets/resources/pr2/urdf/pr2.urdf (robot description, URDF)
Before this commit: robot pr2, 16 links, 15 joints
Links:
- link r_gripper_palm_link: geometry collision box size=0.125 0.095 0.065; visual mesh filename=package://pr2_description/meshes/gripper_v0/gripper_palm.dae

Commit message: pr2 urdf, small stuff

File: ocs2_robotic_assets/resources/pr2/urdf/pr2.urdf (robot description, URDF)
Before this commit: robot pr2, 16 links, 15 joints
Links:
- added link l_elbow_flex_link, mass 1.90327; visual mesh filename=package://pr2_description/meshes/upper_arm_v0/elbow_flex.dae
- added link l_forearm_link, mass 2.57968; collision box size=0.21 0.075 0.075; visual mesh filename=package://pr2_description/meshes/forearm_v0/forearm.dae
- added link l_forearm_roll_link, mass 0.1; visual mesh filename=package://pr2_description/meshes/upper_arm_v0/forearm_roll.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
- added link l_gripper_l_finger_link, mass 0.17126; visual mesh filename=package://pr2_description/meshes/gripper_v0/l_finger.dae
- added link l_gripper_palm_link, mass 0.58007; collision box size=0.125 0.095 0.065; visual mesh filename=package://pr2_description/meshes/gripper_v0/gripper_palm.dae
- added link l_gripper_r_finger_link, mass 0.17389; visual mesh filename=package://pr2_description/meshes/gripper_v0/l_finger.dae
- added link l_shoulder_lift_link, mass 2.74988; visual mesh filename=package://pr2_description/meshes/shoulder_v0/shoulder_lift.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
- added link l_shoulder_pan_link, mass 25.799322; visual mesh filename=package://pr2_description/meshes/shoulder_v0/shoulder_pan.d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
- added link l_upper_arm_link, mass 6.01769; visual mesh filename=package://pr2_description/meshes/upper_arm_v0/upper_arm.dae
- added link l_upper_arm_roll_link, mass 0.1; visual mesh filename=package://pr2_description/meshes/shoulder_v0/upper_arm_roll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
- added link l_wrist_flex_link, mass 0.61402; visual mesh filename=package://pr2_description/meshes/forearm_v0/wrist_flex.dae
- added link l_wrist_roll_link, mass 0.1; visual mesh filename=package://pr2_description/meshes/forearm_v0/wrist_roll.stl
Joints:
- added joint l_elbow_flex_joint: type fixed, parent l_upper_arm_link, child l_elbow_flex_link, origin xyz=0.4 0 0 rpy=0 0 0, axis 0 1 0, limit lower=-2.3213 upper=0.00 effort=30 velocity=3.3
- added joint l_forearm_joint: type fixed, parent l_forearm_roll_link, child l_forearm_link, origin xyz=0 0 0 rpy=0 0 0
- added joint l_forearm_roll_joint: type fixed, parent l_elbow_flex_link, child l_forearm_roll_link, origin xyz=0 0 0 rpy=0 0 0, axis 1 0 0, limit effort=30 velocity=3.6
- added joint l_gripper_l_finger_joint: type fixed, parent l_gripper_palm_link, child l_gripper_l_finger_link, origin xyz=0.07691 0.01 0 rpy=0 0 0, axis 0 0 1, limit lower=0.0 upper=0.548 effort=1000.0 velocity=0.5
- added joint l_gripper_palm_joint: type fixed, parent l_wrist_roll_link, child l_gripper_palm_link, origin xyz=0 0 0 rpy=0 0 0
- added joint l_gripper_r_finger_joint: type fixed, parent l_gripper_palm_link, child l_gripper_r_finger_link, origin xyz=0.07691 -0.01 0 rpy=0 0 0, axis 0 0 -1, limit lower=0.0 upper=0.548 effort=1000.0 velocity=0.5, mimic joint=l_gripper_l_finger_joint multiplier=1 offset=0
- added joint l_shoulder_lift_joint: type fixed, parent l_shoulder_pan_link, child l_shoulder_lift_link, origin xyz=0.1 0 0 rpy=0 0 0, axis 0 1 0, limit lower=-0.5236 upper=1.3963 effort=30 velocity=2.082
- added joint l_shoulder_pan_joint: type fixed, parent torso_lift_link, child l_shoulder_pan_link, origin xyz=0.0 0.188 0.0 rpy=0 0 0, axis 0 0 1, limit lower=-0.714601836603 upper=2.2853981634 effort=30 velocity=2.088
- added joint l_upper_arm_joint: type fixed, parent l_upper_arm_roll_link, child l_upper_arm_link, origin xyz=0 0 0 rpy=0 0 0
- added joint l_upper_arm_roll_joint: type fixed, parent l_shoulder_lift_link, child l_upper_arm_roll_link, origin xyz=0 0 0 rpy=0 0 0, axis 1 0 0, limit lower=-0.8 upper=3.9 effort=30 velocity=3.27
- added joint l_wrist_flex_joint: type fixed, parent l_forearm_link, child l_wrist_flex_link, origin xyz=0.321 0 0 rpy=0 0 0, axis 0 1 0, limit lower=-2.18 upper=0.0 effort=10 velocity=3.078
- added joint l_wrist_roll_joint: type fixed, parent l_wrist_flex_link, child l_wrist_roll_link, origin xyz=0 0 0 rpy=0 0 0, axis 1 0 0, limit effort=10 velocity=3.6
- joint r_forearm_roll_joint: type continuous -> revolute

Commit message: add pr2 wheels to urdf

File: ocs2_robotic_assets/resources/pr2/urdf/pr2.urdf (robot description, URDF)
Before this commit: robot pr2, 28 links, 27 joints
Links:
- added link bl_caster_l_wheel_link, mass 0.44036; collision cylinder length=0.034 radius=0.074792; visual mesh filename=package://pr2_description/meshes/base_v0/wheel.dae
- added link bl_caster_r_wheel_link, mass 0.44036; collision cylinder length=0.034 radius=0.074792; visual mesh filename=package://pr2_description/meshes/base_v0/wheel.dae
- added link bl_caster_rotation_link, mass 3.473082; collision mesh filename=package://pr2_description/meshes/base_v0/caster_L.stl; visual mesh filename=package://pr2_description/meshes/base_v0/caster.stl
- added link br_caster_l_wheel_link, mass 0.44036; collision cylinder length=0.034 radius=0.074792; visual mesh filename=package://pr2_description/meshes/base_v0/wheel.dae
- added link br_caster_r_wheel_link, mass 0.44036; collision cylinder length=0.034 radius=0.074792; visual mesh filename=package://pr2_description/meshes/base_v0/wheel.dae
- added link br_caster_rotation_link, mass 3.473082; collision mesh filename=package://pr2_description/meshes/base_v0/caster_L.stl; visual mesh filename=package://pr2_description/meshes/base_v0/caster.stl
- added link fl_caster_l_wheel_link, mass 0.44036; collision cylinder length=0.034 radius=0.074792; visual mesh filename=package://pr2_description/meshes/base_v0/wheel.dae
- added link fl_caster_r_wheel_link, mass 0.44036; collision cylinder length=0.034 radius=0.074792; visual mesh filename=package://pr2_description/meshes/base_v0/wheel.dae
- added link fl_caster_rotation_link, mass 3.473082; collision mesh filename=package://pr2_description/meshes/base_v0/caster_L.stl; visual mesh filename=package://pr2_description/meshes/base_v0/caster.stl
- added link fr_caster_l_wheel_link, mass 0.44036; collision cylinder length=0.034 radius=0.074792; visual mesh filename=package://pr2_description/meshes/base_v0/wheel.dae
- added link fr_caster_r_wheel_link, mass 0.44036; collision cylinder length=0.034 radius=0.074792; visual mesh filename=package://pr2_description/meshes/base_v0/wheel.dae
- added link fr_caster_rotation_link, mass 3.473082; collision mesh filename=package://pr2_description/meshes/base_v0/caster_L.stl; visual mesh filename=package://pr2_description/meshes/base_v0/caster.stl
Joints:
- added joint bl_caster_l_wheel_joint: type fixed, parent bl_caster_rotation_link, child bl_caster_l_wheel_link, origin xyz=0 0.049 0 rpy=0 0 0, axis 0 1 0, limit effort=25 velocity=15
- added joint bl_caster_r_wheel_joint: type fixed, parent bl_caster_rotation_link, child bl_caster_r_wheel_link, origin xyz=0 -0.049 0 rpy=0 0 0, axis 0 1 0, limit effort=25 velocity=15
- added joint bl_caster_rotation_joint: type fixed, parent base_link, child bl_caster_rotation_link, origin xyz=-0.2246 0.2246 0.0282 rpy=0 0 0, axis 0 0 1, limit effort=25.0 velocity=10
- added joint br_caster_l_wheel_joint: type fixed, parent br_caster_rotation_link, child br_caster_l_wheel_link, origin xyz=0 0.049 0 rpy=0 0 0, axis 0 1 0, limit effort=25 velocity=15
- added joint br_caster_r_wheel_joint: type fixed, parent br_caster_rotation_link, child br_caster_r_wheel_link, origin xyz=0 -0.049 0 rpy=0 0 0, axis 0 1 0, limit effort=25 velocity=15
- added joint br_caster_rotation_joint: type fixed, parent base_link, child br_caster_rotation_link, origin xyz=-0.2246 -0.2246 0.0282 rpy=0 0 0, axis 0 0 1, limit effort=25.0 velocity=10
- added joint fl_caster_l_wheel_joint: type fixed, parent fl_caster_rotation_link, child fl_caster_l_wheel_link, origin xyz=0 0.049 0 rpy=0 0 0, axis 0 1 0, limit effort=25 velocity=15
- added joint fl_caster_r_wheel_joint: type fixed, parent fl_caster_rotation_link, child fl_caster_r_wheel_link, origin xyz=0 -0.049 0 rpy=0 0 0, axis 0 1 0, limit effort=25 velocity=15
- added joint fl_caster_rotation_joint: type fixed, parent base_link, child fl_caster_rotation_link, origin xyz=0.2246 0.2246 0.0282 rpy=0 0 0, axis 0 0 1, limit effort=25.0 velocity=10
- added joint fr_caster_l_wheel_joint: type fixed, parent fr_caster_rotation_link, child fr_caster_l_wheel_link, origin xyz=0 0.049 0 rpy=0 0 0, axis 0 1 0, limit effort=25 velocity=15
- added joint fr_caster_r_wheel_joint: type fixed, parent fr_caster_rotation_link, child fr_caster_r_wheel_link, origin xyz=0 -0.049 0 rpy=0 0 0, axis 0 1 0, limit effort=25 velocity=15
- added joint fr_caster_rotation_joint: type fixed, parent base_link, child fr_caster_rotation_link, origin xyz=0.2246 -0.2246 0.0282 rpy=0 0 0, axis 0 0 1, limit effort=25.0 velocity=10

Commit message: small updates, hsr WIP

File: ocs2_robotic_assets/resources/pr2/urdf/pr2.urdf (robot description, URDF)
Before this commit: robot pr2, 40 links, 39 joints
Links:
- link l_forearm_link: geometry collision box size=0.15 0.075 0.075; visual mesh filename=package://pr2_description/meshes/forearm_v0/forearm.dae
- link r_forearm_link: geometry collision box size=0.15 0.075 0.075; visual mesh filename=package://pr2_description/meshes/forearm_v0/forearm.dae

Commit message: mpc_mrt node working

File: ocs2_robotic_assets/resources/pr2/urdf/pr2.urdf (robot description, URDF)
Before this commit: robot pr2, 40 links, 39 joints
Links:
- added link base_bellow_link, mass 1.0; collision box size=0.05 0.37 0.3; visual box size=0.05 0.37 0.3
- added link base_footprint, mass 1.0; collision box size=0.001 0.001 0.001; visual box size=0.01 0.01 0.01
Joints:
- added joint base_bellow_joint: type fixed, parent base_link, child base_bellow_link, origin xyz=-0.29 0 0.8 rpy=0 0 0
- added joint base_footprint_joint: type fixed, parent base_footprint, child base_link, origin xyz=0 0 0.051 rpy=0 0 0
